File: pcb/bb-8.sch (EAGLE design)
At the start: 24 parts, among them T1 2N2222, X1 STEREOJACK

Commit message: Squashed commit of the following:
commit c327650e5103bb6a6949c6a1538a163dea4dba5a
Author: Patrick Ryan <pat.m.ryan@gmail.com>
Date:   Sat Aug 20 09:49:49 2022 -0400

    Updates to PCB

commit 971e034c2edcb3dc5db781baa092387508605f21
Author: Patrick Ryan <pat.m.ryan@gmail.com>
Date:   Sat Aug 20 09:49:32 2022 -0400

    Splitting up main drive into separate files

commit 5c3a9991173692b4d5a5e5dc78048e5e86c772e9
Author: Patrick Ryan <pat.m.ryan@gmail.com>
Date:   Fri Jul 1 13:35:34 2022 -0400

    Splitting up drive functions into separate files
Parts:
- removed 7.2V: 1X2-3.5MM, adafruit:1X2-3.5MM
- removed SERVO1, SERVO2: (no value), pinhead:PINHD-1X3
- removed U$4, U$5: KEYSTONE_3568, BB8:KEYSTONE_3568
- added 12V, 7V2: 1X2-3.5MM, adafruit:1X2-3.5MM
- added IC1: 786TV, linear:786TV
- added JP2: (no value), pinhead:PINHD-1X4
- added JP3, JP4: (no value), pinhead:PINHD-1X8
Connections:
- removed net N$20: 5V.1, U$4.2A
- removed net N$21: 7.2V.1, U$5.2A
- new net +12V: 12V.1, IC1.VI, JP3.1, JP4.1, SBUS.2
- new net 5V_RAW: IC1.VO, R2.2
- net +5V: now also 5V.1, JP2.1, JP3.2, JP3.3, JP4.2, JP4.3; no longer R2.2, SBUS.2, U$4.1A
- net +7V: now also 7V2.1, JP3.4, JP4.4; no longer SERVO1.2, SERVO2.2, U$5.1A
- net GND: now also 12V.2, 7V2.2, IC1.GND, JP2.4, JP3.5, JP3.6, JP3.7, JP3.8, JP4.5, JP4.6, JP4.7, JP4.8; no longer 7.2V.2, SERVO1.3, SERVO2.3
- net SCL: now also JP2.3
- net SDA: now also JP2.2
- net SERVO_1: no longer SERVO1.1
- net SERVO_2: no longer SERVO2.1
Other:
- note added: "5V Regulator"
- note added: "Body LEDs"
- note added: "Power Expander"
- note added: "Servo PWM"
- note added: "V Batt"
- note removed: "Left Servo"
- note removed: "Right Servo"
- moved on the sheet: BODYLIGHTS, DOME_POT, FLY, JP1, MAIN, R1, R2, R3, S2S, S2S_POT, SBUS, T1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

Commit message: Updates to board
Parts:
- removed 12V: 1X2-3.5MM, adafruit:1X2-3.5MM
- removed IC1: 786TV, linear:786TV
- removed JP1: (no value), pinhead:PINHD-1X3
- removed JP2: (no value), pinhead:PINHD-1X4
- removed JP3, JP4: (no value), pinhead:PINHD-1X8
- added C1: 0.22uF, rcl:C-EU050-024X044
Connections:
- removed net +12V: 12V.1, IC1.VI, JP3.1, JP4.1, SBUS.2
- removed net 5V_RAW: IC1.VO, R2.2
- removed net SERVO_1: U$7.5
- removed net SERVO_2: U$7.4
- net +5V: now also R2.2; no longer JP2.1, JP3.2, JP3.3, JP4.2, JP4.3
- net +7V: now also SBUS.2; no longer JP3.4, JP4.4
- net DAC_R: no longer JP1.3
- net GND: now also C1.2; no longer 12V.2, IC1.GND, JP1.2, JP2.4, JP3.5, JP3.6, JP3.7, JP3.8, JP4.5, JP4.6, JP4.7, JP4.8
- net N$6: no longer JP1.1
- net S2S_POT: now also C1.1
- net SCL: no longer JP2.3
- net SDA: no longer JP2.2
Other:
- note removed: "5V Regulator"
- note removed: "Power Expander"
- note removed: "Servo PWM"
- note removed: "V Batt"
- moved on the sheet: BODYLIGHTS, DOME_POT, R1, R2, R3, S2S_POT, SBUS, T1, X1
